File: 86_BOX_PANEL.kicad_pcb (KiCad board)
At the start: 2 copper layers, 60 x 47.5 mm, 48 parts, among them J1 Conn_01x01_Socket, J2 Conn_01x01_Socket, J3 Conn_01x01_Socket, J4 Conn_01x01_Socket, J5 Conn_01x01_Socket, J6 Conn_01x01_Socket, J7 Conn_01x04_Pin, SW1 SW_Push, SW2 SW_Push, U1 HLK_5V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

Commit message: nc
Parts:
- ESP1: footprint footprint:ESP32-SOLO-1 -> YZ-ICs:ESP32-SOLO-1
- FL1: footprint footprint:UU9.8 -> YZ-PWR:UU9.8
- J1, J4: footprint footprint:springNeedle -> YZ-PWR:springNeedle
- J2, J3, J5, J6: footprint footprint:BlockTerminal -> YZ-Connector:BlockTerminal
- U1: footprint footprint:HLK-10M05 -> YZ-PWR:HLK-10M05
Connections:
- ESP1 pad P$39: GND -> (no net)
