File: 86_BOX_PANEL.kicad_sch (KiCad schematic)
At the start: 46 parts, among them J1 Conn_01x01_Socket, J2 Conn_01x01_Socket, J3 Conn_01x01_Socket, J4 Conn_01x01_Socket, J5 Conn_01x01_Socket, J6 Conn_01x01_Socket, J7 Conn_01x04_Pin, SW1 SW_Push, SW2 SW_Push, U1 HLK_5V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

Commit message: nc
Parts:
- ESP1: footprint footprint:ESP32-SOLO-1 -> YZ-ICs:ESP32-SOLO-1; symbol ESP32-SOLO-1:ESP32-SOLO-1 -> YZ_ICs:ESP32-SOLO-1
- FL1: footprint footprint:UU9.8 -> YZ-PWR:UU9.8
- J1, J4: footprint footprint:springNeedle -> YZ-PWR:springNeedle
- J2, J3, J5, J6: footprint footprint:BlockTerminal -> YZ-Connector:BlockTerminal
- U1: footprint footprint:HLK-10M05 -> YZ-PWR:HLK-10M05; symbol 86box:HLK-10M05 -> YZ_Library:HLK-10M05
Connections:
- net GND: no longer ESP1.P$39 (GND4)
Changed lines of the file:
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@@
       (effects (font (size 1.27 1.27)))
     )
-    (property "Footprint" "footprint:springNeedle" (at 22.86 73.66 0)
+    (property "Footprint" "YZ-PWR:springNeedle" (at 22.86 73.66 0)
       (effects (font (size 1.27 1.27)) hide)
     )
@@
       (effects (font (size 1.27 1.27)))
     )
-    (property "Footprint" "footprint:BlockTerminal" (at 162.56 64.77 0)
+    (property "Footprint" "YZ-Connector:BlockTerminal" (at 162.56 64.77 0)
       (effects (font (size 1.27 1.27)) hide)
     )
@@
       (effects (font (size 1.27 1.27)))
     )
-    (property "Footprint" "footprint:BlockTerminal" (at 162.56 67.31 0)
+    (property "Footprint" "YZ-Connector:BlockTerminal" (at 162.56 67.31 0)
       (effects (font (size 1.27 1.27)) hide)
     )
@@
     )
   )
-  (symbol (lib_id "ESP32-SOLO-1:ESP32-SOLO-1") (at 99.06 148.59 0) (unit 1)
+  (symbol (lib_id "YZ_ICs:ESP32-SOLO-1") (at 99.06 148.59 0) (unit 1)
     (in_bom yes) (on_board yes) (dnp no) (fields_autoplaced)
     (property "Reference" "ESP1" (at 100.33 118.11 0)
@@
       (effects (font (size 1.27 1.27)))
     )
-    (property "Footprint" "footprint:ESP32-SOLO-1" (at 99.06 148.59 0)
+    (property "Footprint" "YZ-ICs:ESP32-SOLO-1" (at 99.06 148.59 0)
       (effects (font (size 1.27 1.27)) (justify bottom) hide)
     )
@@
     (pin "P$8")
     (pin "P$9")
-    (pin "P$39")
     (instances
       (project "86_BOX_PANEL"
@@
       (effects (font (size 1.27 1.27)))
     )
-    (property "Footprint" "footprint:springNeedle" (at 27.94 85.09 0)
+    (property "Footprint" "YZ-PWR:springNeedle" (at 27.94 85.09 0)
       (effects (font (size 1.27 1.27)) hide)
     )
@@
       (effects (font (size 1.27 1.27)))
     )
-    (property "Footprint" "footprint:BlockTerminal" (at 31.75 35.56 0)
-      (effects (font (size 1.27 1.27)) hide)
+    (property "Footprint" "YZ-Connector:BlockTerminal" (at 31.75 35.56 0)
+      (effects (font (size 1.27 1.27)))
     )
     (property "Datasheet" "~" (at 31.75 35.56 0)
@@
     )
   )
-  (symbol (lib_id "86box:HLK-10M05") (at 82.55 40.64 0) (unit 1)
+  (symbol (lib_id "YZ_Library:HLK-10M05") (at 82.55 40.64 0) (unit 1)
     (in_bom yes) (on_board yes) (dnp no)
     (property "Reference" "U1" (at 98.425 27.94 0)
@@
       (effects (font (size 1.27 1.27)) (justify left))
     )
-    (property "Footprint" "footprint:HLK-10M05" (at 96.52 33.02 0)
+    (property "Footprint" "YZ-PWR:HLK-10M05" (at 96.52 33.02 0)
       (effects (font (size 1.27 1.27)) hide)
     )
@@
       (effects (font (size 1.27 1.27)))
     )
-    (property "Footprint" "footprint:BlockTerminal" (at 31.75 33.02 0)
+    (property "Footprint" "YZ-Connector:BlockTerminal" (at 31.75 33.02 0)
       (effects (font (size 1.27 1.27)) hide)
     )
@@
       (effects (font (size 1.27 1.27)))
     )
-    (property "Footprint" "footprint:UU9.8" (at 78.74 33.274 0)
-      (effects (font (size 1.27 1.27)) hide)
-    )
+    (property "Footprint" "YZ-PWR:UU9.8" (at 78.74 33.274 0)
+      (effects (font (size 1.27 1.27)) hide)
+    )
